File: RPico.kicad_sch (KiCad schematic)
At the start: 35 parts, among them IC2 W25Q128JVSIQ, IC3 AMS1117-3.3, J10 USB_C_Receptacle_USB2.0_16P, J5 S3B-ZR-SM4A-TF, SW1 BOOTSEL, SW2 RESET, U4 RP2040, Y2 Crystal_GND24_Small

Commit message: modify
Parts:
- removed C34, C35, C36: 10uF, Capacitor_SMD:C_0603_1608Metric, symbol Device:C
- removed C37, C38, C39, C40, C41, C42, C43, C44, C46, C47, C49: 100nF, Capacitor_SMD:C_0603_1608Metric, symbol Device:C
- removed C45, C48: 1uF, Capacitor_SMD:C_0603_1608Metric, symbol Device:C
- removed C50, C51: 18pF, Capacitor_SMD:C_0603_1608Metric, symbol Device:C
- removed D9: LED_GREEN, LED_SMD:LED_0603_1608Metric, symbol Device:LED
- removed H1: SWCLK, Connector_Pin:Pin_D1.0mm_L10.0mm, symbol Mechanical:MountingHole_Pad
- removed H2: SWD, Connector_Pin:Pin_D1.0mm_L10.0mm, symbol Mechanical:MountingHole_Pad
- removed IC2: W25Q128JVSIQ, SamaSys_Parts:SOIC127P790X216-8N, symbol SamacSys_Parts:W25Q128JVSIQ
- removed IC3: AMS1117-3.3, SamaSys_Parts:SOT229P700X180-4N, symbol SamacSys_Parts:AMS1117-3.3
- removed J10: USB_C_Receptacle_USB2.0_16P, Connector_USB:USB_C_Receptacle_GCT_USB4105-xx-A_16P_TopMnt_Horizontal, symbol Connector:USB_C_Receptacle_USB2.0_16P
- removed J5: S3B-ZR-SM4A-TF, SamaSys_Parts:S3BZRSM4ATFLF, symbol SamacSys_Parts:S3B-ZR-SM4A-TF
- removed R14, R15: 5.1k, Resistor_SMD:R_0603_1608Metric, symbol Device:R
- removed R16, R17: 27, Resistor_SMD:R_0603_1608Metric, symbol Device:R
- removed R18: 470, Resistor_SMD:R_0603_1608Metric, symbol Device:R
- removed SW1: BOOTSEL, Button_Switch_SMD:SW_Push_1P1T_NO_Vertical_Wuerth_434133025816, symbol Switch:SW_Push
- removed SW2: RESET, Button_Switch_SMD:SW_Push_1P1T_NO_Vertical_Wuerth_434133025816, symbol Switch:SW_Push
- removed TP1: TestPoint, TestPoint:TestPoint_Pad_2.0x2.0mm, symbol Connector:TestPoint
- removed U4: RP2040, Package_DFN_QFN:QFN-56-1EP_7x7mm_P0.4mm_EP3.2x3.2mm, symbol MCU_RaspberryPi:RP2040
- removed Y2: Crystal_GND24_Small, Crystal:Crystal_SMD_0603-4Pin_6.0x3.5mm, symbol Device:Crystal_GND24_Small
Connections:
- no-connect marks 17 -> 0
Other:
- note removed: "50pinがない.DVDD,1.1V"
- note removed: "QSPI FLASH"
