File: ethernet.kicad_sch (KiCad schematic)
At the start: 40 parts, among them J1 S4B-ZR-SM4A-TF_LF_, J2 S4B-ZR-SM4A-TF_LF_, J3 S4B-ZR-SM4A-TF_LF_, J4 S4B-ZR-SM4A-TF_LF_, T1 H1102NL, T2 H1102NL, T3 H1102NL, T4 H1102NL

Commit message: modify
Parts:
- removed C18, C19, C20, C21, C24, C28, C32: 0.1uF, Capacitor_SMD:C_0603_1608Metric, symbol Device:C
- removed D1, D2, D3, D4, D5, D6, D7, D8: LED, LED_SMD:LED_0603_1608Metric, symbol Device:LED
- removed J1, J2, J3, J4: S4B-ZR-SM4A-TF_LF_, SamaSys_Parts:S4BZRSM4ATFLF, symbol SamacSys_Parts:S4B-ZR-SM4A-TF_LF_
- removed T1: H1102NL, SamaSys_Parts:SOIC127P940X597-16N, symbol SamacSys_Parts:H1102NL
- added FB6: HI1206N101R-00, SamaSys_Parts:BEADC3216X130N, symbol SamacSys_Parts:HI1206N101R-00
- added J1: Conn_02x04_Top_Bottom, me:PinSocket_2x04_P2.54mm_Horizontal, symbol Connector_Generic:Conn_02x04_Top_Bottom
- added J3: Conn_02x05_Top_Bottom, me:PinSocket_2x05_P2.54mm_Horizontal, symbol Connector_Generic:Conn_02x05_Top_Bottom
- added LED1: SPD_2, SamaSys_Parts:LEDC1608X70N, symbol SamacSys_Parts:KT-0603R
- added LED10: LK_AK_4, SamaSys_Parts:LEDC1608X70N, symbol SamacSys_Parts:KT-0805G
- added LED2: SPD_1, SamaSys_Parts:LEDC1608X70N, symbol SamacSys_Parts:KT-0603R
- added LED5: SPD_3, SamaSys_Parts:LEDC1608X70N, symbol SamacSys_Parts:KT-0603R
- added LED6: SPD_4, SamaSys_Parts:LEDC1608X70N, symbol SamacSys_Parts:KT-0603R
- added LED7: LK_AK_2, SamaSys_Parts:LEDC1608X70N, symbol SamacSys_Parts:KT-0805G
- added LED8: LK_AK_1, SamaSys_Parts:LEDC1608X70N, symbol SamacSys_Parts:KT-0805G
- added LED9: LK_AK_3, SamaSys_Parts:LEDC1608X70N, symbol SamacSys_Parts:KT-0805G
- added R16, R17, R18: 75, Resistor_SMD:R_0603_1608Metric, symbol Device:R
- C25, C29, C33: value 0.1uF -> 1nF/2kV; footprint Capacitor_SMD:C_0603_1608Metric -> Capacitor_SMD:C_1206_3216Metric
Connections:
- net GND: now also FB6.1, J3.10 (Pin_10), J3.5 (Pin_5); no longer C25.2, C29.2, C33.2
- net RXM1: now also J3.4 (Pin_4)
- net RXP1: now also J3.3 (Pin_3)
- net TXM1: now also J3.2 (Pin_2)
- net TXP1: now also J3.1 (Pin_1)
- net VDDIO: now also LED1.2 (A), LED10.1 (A), LED2.2 (A), LED5.2 (A), LED6.2 (A), LED7.1 (A), LED8.1 (A), LED9.1 (A)
- net at T3.10 (NC_3): now also T3.15 (NC_6), R17.1
- net at T3.11 (RX+): now also J3.8 (Pin_8)
- net at T3.14 (TX-): now also J3.7 (Pin_7)
- net at C29.1: now also R17.2; no longer T3.15 (NC_6)
- net at T3.16 (TX+): now also J3.6 (Pin_6)
- net at T3.9 (RX-): now also J3.9 (Pin_9)
- net at R11.2: now also LED9.2 (K)
- net at R9.2: now also LED8.2 (K)
- net at R8.2: now also LED2.1 (K)
- net at T4.10 (NC_3): now also T4.15 (NC_6), R18.1
- net at R12.2: now also LED6.1 (K)
- net at T2.16 (TX+): now also J1.1 (Pin_1)
- net at T2.14 (TX-): now also J1.2 (Pin_2)
- net at T2.11 (RX+): now also J1.3 (Pin_3)
- net at T2.9 (RX-): now also J1.4 (Pin_4)
- net at R10.2: now also LED5.1 (K)
- net at R13.2: now also LED10.2 (K)
- net at R7.2: now also LED7.2 (K)
- net at T2.10 (NC_3): now also T2.15 (NC_6), R16.1
- net at C25.1: now also R16.2; no longer T2.15 (NC_6)
- net at C33.1: now also R18.2; no longer T4.15 (NC_6)
- net at T4.16 (TX+): now also J1.5 (Pin_5)
- net at T4.14 (TX-): now also J1.6 (Pin_6)
- net at T4.11 (RX+): now also J1.7 (Pin_7)
- net at T4.9 (RX-): now also J1.8 (Pin_8)
- net at R6.2: now also LED1.1 (K)
- new net GNDS: C25.2, C29.2, C33.2, FB6.2
- no-connect marks 24 -> 12
Other:
- note added: "palse transformerがRJ45に内蔵されているので H1102NLは不要"
- note removed: "Link/Act"
- note removed: "Speed"
- moved on the sheet: C29, C33, R10, R11, R12, R13, R6, R7, R8, R9
