File: zz_micro_l2sw.kicad_pcb (KiCad board)
At the start: 2 copper layers, 31 x 100.5 mm, 135 parts, among them IC1 KSZ8795CLXIC, IC2 W25Q128JVSIQ, IC3 AMS1117-3.3, IC4 MIC5309-1.2YD6, J1 S4B-ZR-SM4A-TF_LF_, J10 USB_C_Receptacle_USB2.0_16P, J2 S4B-ZR-SM4A-TF_LF_, J3 S4B-ZR-SM4A-TF_LF_, J4 S4B-ZR-SM4A-TF_LF_, J5 S3B-ZR-SM4A-TF, SW1 BOOTSEL, SW2 RESET, T1 H1102NL, T2 H1102NL, T3 H1102NL, T4 H1102NL, U4 RP2040, Y2 Crystal_GND24_Small, Y3 25MHz

Commit message: modify
Parts:
- removed C18, C19, C20, C21, C24, C28, C32: 0.1uF, Capacitor_SMD:C_0603_1608Metric
- removed C34, C35, C36: 10uF, Capacitor_SMD:C_0603_1608Metric
- removed C37, C38, C39, C40, C41, C42, C43, C44, C46, C47, C49: 100nF, Capacitor_SMD:C_0603_1608Metric
- removed C45, C48: 1uF, Capacitor_SMD:C_0603_1608Metric
- removed C50, C51: 18pF, Capacitor_SMD:C_0603_1608Metric
- removed D1, D2, D3, D4, D5, D6, D7, D8: LED, LED_SMD:LED_0603_1608Metric
- removed D9: LED_GREEN, LED_SMD:LED_0603_1608Metric
- removed H1: SWCLK, Connector_Pin:Pin_D1.0mm_L10.0mm
- removed H2: SWD, Connector_Pin:Pin_D1.0mm_L10.0mm
- removed IC2: W25Q128JVSIQ, SamaSys_Parts:SOIC127P790X216-8N
- removed IC3: AMS1117-3.3, SamaSys_Parts:SOT229P700X180-4N
- removed J10: USB_C_Receptacle_USB2.0_16P, Connector_USB:USB_C_Receptacle_GCT_USB4105-xx-A_16P_TopMnt_Horizontal
- removed J4: S4B-ZR-SM4A-TF_LF_, SamaSys_Parts:S4BZRSM4ATFLF
- removed J5: S3B-ZR-SM4A-TF, SamaSys_Parts:S3BZRSM4ATFLF
- removed R14, R15: 5.1k, Resistor_SMD:R_0603_1608Metric
- removed SW1: BOOTSEL, Button_Switch_SMD:SW_Push_1P1T_NO_Vertical_Wuerth_434133025816
- removed SW2: RESET, Button_Switch_SMD:SW_Push_1P1T_NO_Vertical_Wuerth_434133025816
- removed T1: H1102NL, SamaSys_Parts:SOIC127P940X597-16N
- removed TP1: TestPoint, TestPoint:TestPoint_Pad_2.0x2.0mm
- removed U4: RP2040, Package_DFN_QFN:QFN-56-1EP_7x7mm_P0.4mm_EP3.2x3.2mm
- removed Y2: Crystal_GND24_Small, Crystal:Crystal_SMD_0603-4Pin_6.0x3.5mm
- removed Y3: 25MHz, Crystal:Crystal_SMD_0603-4Pin_6.0x3.5mm
- added C1: 100nF, Capacitor_SMD:C_0603_1608Metric, F.Cu at (205.6, 95.2)
- added C10: 100nF, Capacitor_SMD:C_0603_1608Metric, F.Cu at (217.8, 90.4)
- added C11: 100nF, Capacitor_SMD:C_0603_1608Metric, F.Cu at (217.8, 91.9)
- added C12: 100nF, Capacitor_SMD:C_0603_1608Metric, F.Cu at (217.8, 93.4)
- added C13: 100nF, Capacitor_SMD:C_0603_1608Metric, F.Cu at (217.8, 84.4)
- added C14: 100nF, Capacitor_SMD:C_0603_1608Metric, F.Cu at (217.8, 82.9)
- added C15: 10uF, Capacitor_SMD:C_0603_1608Metric, F.Cu at (214.5, 80.2)
- added C16: 10uF, Capacitor_SMD:C_0603_1608Metric, F.Cu at (211.5, 80.2)
- added C17: 10uF, Capacitor_SMD:C_0603_1608Metric, F.Cu at (208.5, 80.2)
- added C2: 100nF, Capacitor_SMD:C_0603_1608Metric, F.Cu at (205.6, 96.7)
- added C3: 1uF, Capacitor_SMD:C_0603_1608Metric, F.Cu at (205.6, 93.7)
- added C4: 100nF, Capacitor_SMD:C_0603_1608Metric, F.Cu at (230.5, 93.2)
- added C5: 1uF, Capacitor_SMD:C_0603_1608Metric, F.Cu at (217.8, 87.4)
- added C6: 100nF, Capacitor_SMD:C_0603_1608Metric, F.Cu at (217.8, 85.9)
- added C7: 18pF, Capacitor_SMD:C_0603_1608Metric, F.Cu at (210.4, 97.0)
- added C8: 100nF, Capacitor_SMD:C_0603_1608Metric, F.Cu at (217.7, 88.9)
- added C86: 100nF, Capacitor_SMD:C_0603_1608Metric, F.Cu at (224.6, 107.3)
- added C9: 18pF, Capacitor_SMD:C_0603_1608Metric, F.Cu at (210.4, 104.2)
- added FB6: HI1206N101R-00, SamaSys_Parts:BEADC3216X130N, F.Cu at (213.0, 133.2)
- added IC5: RP2040, SamaSys_Parts:QFN40P700X700X90-57N-D, F.Cu at (219.6, 101.2)
- added IC7: W25Q128JVSIQ, SamaSys_Parts:SOIC127P790X216-8N, F.Cu at (228.3, 100.7)
- added LED1: SPD_2, SamaSys_Parts:LEDC1608X70N, F.Cu at (202.0, 138.3)
- added LED10: LK_AK_4, SamaSys_Parts:LEDC1608X70N, F.Cu at (217.7, 141.7)
- added LED2: SPD_1, SamaSys_Parts:LEDC1608X70N, F.Cu at (202.0, 144.9)
- added LED3: PICO, SamaSys_Parts:KT0805G, F.Cu at (217.8, 78.0)
- added LED4: PWR, SamaSys_Parts:LEDC1608X70N, F.Cu at (206.6, 82.9)
- added LED5: SPD_3, SamaSys_Parts:LEDC1608X70N, F.Cu at (217.7, 144.9)
- added LED6: SPD_4, SamaSys_Parts:LEDC1608X70N, F.Cu at (217.7, 138.3)
- added LED7: LK_AK_2, SamaSys_Parts:LEDC1608X70N, F.Cu at (202.0, 141.6)
- added LED8: LK_AK_1, SamaSys_Parts:LEDC1608X70N, F.Cu at (202.0, 148.2)
- added LED9: LK_AK_3, SamaSys_Parts:LEDC1608X70N, F.Cu at (217.7, 148.2)
- added R1: 5.1k, Resistor_SMD:R_0603_1608Metric, F.Cu at (220.3, 79.6)
- added R2: 27, Resistor_SMD:R_0603_1608Metric, F.Cu at (224.6, 101.4)
- added R27: 470, Resistor_SMD:R_0603_1608Metric, F.Cu at (217.8, 81.3)
- added R3: 27, Resistor_SMD:R_0603_1608Metric, F.Cu at (224.6, 104.3)
- added R4: 5.1k, Resistor_SMD:R_0603_1608Metric, F.Cu at (220.3, 83.1)
- added R5: 470, Resistor_SMD:R_0603_1608Metric, F.Cu at (206.5, 86.4)
- added S1: RESET, SamaSys_Parts:TS1088AR02016, F.Cu at (228.6, 87.9)
- added S2: BOOTSEL, SamaSys_Parts:TS1088AR02016, F.Cu at (223.7, 87.9)
- added U1: TYPE-C 16PIN 2MD(073), me:TYPE-C 16PIN 2MD(073), F.Cu at (226.1, 78.1)
- added Y1: X322525MOB4SI, SamaSys_Parts:X322525MOB4SI, F.Cu at (208.8, 119.1)
- added Y4: 12MHz, SamaSys_Parts:X322512MSB4SI, F.Cu at (210.4, 100.6)
- C25, C29, C33: value 0.1uF -> 1nF/2kV; footprint Capacitor_SMD:C_0603_1608Metric -> Capacitor_SMD:C_1206_3216Metric
- C68, C71, C74, C78, C80, C82: footprint Capacitor_SMD:C_0603_1608Metric -> Capacitor_SMD:C_1206_3216Metric
- J1: value S4B-ZR-SM4A-TF_LF_ -> Conn_02x04_Top_Bottom; footprint SamaSys_Parts:S4BZRSM4ATFLF -> me:PinSocket_2x04_P2.54mm_Horizontal
- J2: value S4B-ZR-SM4A-TF_LF_ -> Conn_01x05; footprint SamaSys_Parts:S4BZRSM4ATFLF -> Connector_PinSocket_2.54mm:PinSocket_1x05_P2.54mm_Vertical
- J3: value S4B-ZR-SM4A-TF_LF_ -> Conn_02x05_Top_Bottom; footprint SamaSys_Parts:S4BZRSM4ATFLF -> me:PinSocket_2x05_P2.54mm_Horizontal; moved to F.Cu
- JP1, JP2, JP3: footprint Jumper:SolderJumper-2_P1.3mm_Bridged2Bar_Pad1.0x1.5mm -> Jumper:SolderJumper-2_P1.3mm_Open_RoundedPad1.0x1.5mm
- R16, R17: value 27 -> 75
- R18: value 470 -> 75
- moved J2 70.2 mm to (213.1, 77.3), turned to -90 degrees
- moved C52 60.9 mm to (203.4, 123.0), turned to 90 degrees
- moved C54 60.0 mm to (201.8, 123.1), turned to -90 degrees
- moved C53 59.0 mm to (201.8, 120.1), turned to 90 degrees
- moved C55 59.0 mm to (201.8, 117.1), turned to -90 degrees
- moved C60 58.7 mm to (205.0, 123.0), turned to -90 degrees
- moved C62 55.9 mm to (204.9, 120.7), turned to 180 degrees
- moved C64 53.8 mm to (204.9, 119.2), turned to 180 degrees
- moved C66 51.7 mm to (204.9, 117.7), turned to 180 degrees
- moved R16 51.0 mm to (230.7, 141.1), turned to 90 degrees
- moved R18 44.4 mm to (230.7, 135.1), turned to -90 degrees
- moved R17 41.8 mm to (201.8, 132.1)
- moved C57 35.8 mm to (229.9, 109.6)
- moved C59 34.5 mm to (229.9, 111.1)
- moved C56 34.5 mm to (229.9, 106.6)
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- renumbered JP6 to JP10, JP9 to JP11, JP8 to JP12, JP10 to JP13, JP5 to JP7, JP4 to JP8, JP7 to JP9
Connections:
- C25 pad 1: Net-(T2-NC_6) -> Net-(C25-Pad1)
- C25 pad 2: GND -> GNDS
- C29 pad 1: Net-(T3-NC_6) -> Net-(C29-Pad1)
- C29 pad 2: GND -> GNDS
- C33 pad 1: Net-(T4-NC_6) -> Net-(C33-Pad1)
- C33 pad 2: GND -> GNDS
- C84 pad 1: KSZ8795_XI -> Net-(Y1-GND_2)
- C85 pad 1: KSZ8795_XO -> Net-(Y1-GND_1)
- IC1 pad 23: INTR_N -> INTR_N_KSZ8795
- IC1 pad 66: SPIQ -> SPI0_RX
- IC1 pad 67: SCL_MDC -> SPI0_SCK
- IC1 pad 68: SDA_MDIO -> SPI0_TX
- IC1 pad 69: SPIS_N -> SPI0_CSn
- IC1 pad 72: RESET_N -> RSTn_KSZ8795
- J1 pad 1: Net-(T1-RX-) -> Net-(J1-Pin_1)
- J1 pad 2: Net-(T1-RX+) -> Net-(J1-Pin_2)
- J1 pad 3: Net-(T1-TX-) -> Net-(J1-Pin_3)
- J1 pad 4: Net-(T1-TX+) -> Net-(J1-Pin_4)
- J1 pad 5: unconnected-(J1-MP1-Pad5) -> Net-(J1-Pin_5)
- J1 pad 6: unconnected-(J1-MP2-Pad6) -> Net-(J1-Pin_6)
- J2 pad 1: Net-(T2-RX-) -> TX0
- J2 pad 2: Net-(T2-RX+) -> RX0
- J2 pad 3: Net-(T2-TX-) -> SWD
- J2 pad 4: Net-(T2-TX+) -> SWCLK
- J2 pad 5: unconnected-(J2-MP1-Pad5) -> GND
- J3 pad 1: Net-(T3-RX-) -> TXP1
- J3 pad 2: Net-(T3-RX+) -> TXM1
- J3 pad 3: Net-(T3-TX-) -> RXP1
- J3 pad 4: Net-(T3-TX+) -> RXM1
- J3 pad 5: unconnected-(J3-MP1-Pad5) -> GND
- J3 pad 6: unconnected-(J3-MP2-Pad6) -> Net-(J3-Pin_6)
- R16 pad 1: D_P -> Net-(T2-NC_3)
- R16 pad 2: Net-(U4-USB_DP) -> Net-(C25-Pad1)
- R17 pad 1: D_N -> Net-(T3-NC_3)
- R17 pad 2: Net-(U4-USB_DM) -> Net-(C29-Pad1)
- R18 pad 1: RP2040_LED -> Net-(T4-NC_3)
- R18 pad 2: Net-(D9-A) -> Net-(C33-Pad1)
- T2 pad 11: Net-(T2-RX+) -> Net-(J1-Pin_3)
- T2 pad 14: Net-(T2-TX-) -> Net-(J1-Pin_2)
- T2 pad 15: Net-(T2-NC_6) -> Net-(T2-NC_3)
- T2 pad 16: Net-(T2-TX+) -> Net-(J1-Pin_1)
- T2 pad 9: Net-(T2-RX-) -> Net-(J1-Pin_4)
- T3 pad 11: Net-(T3-RX+) -> Net-(J3-Pin_8)
- T3 pad 14: Net-(T3-TX-) -> Net-(J3-Pin_7)
- T3 pad 15: Net-(T3-NC_6) -> Net-(T3-NC_3)
- T3 pad 16: Net-(T3-TX+) -> Net-(J3-Pin_6)
- T3 pad 9: Net-(T3-RX-) -> Net-(J3-Pin_9)
- T4 pad 11: Net-(T4-RX+) -> Net-(J1-Pin_7)
- T4 pad 14: Net-(T4-TX-) -> Net-(J1-Pin_6)
- T4 pad 15: Net-(T4-NC_6) -> Net-(T4-NC_3)
- T4 pad 16: Net-(T4-TX+) -> Net-(J1-Pin_5)
- T4 pad 9: Net-(T4-RX-) -> Net-(J1-Pin_8)
Routing:
- net GND: track 107.9 -> 313.8 mm, vias 0 -> 84
- net VDDIO: track 39.8 -> 235.2 mm, vias 2 -> 8
- net VDD12D: track 12.1 -> 122.1 mm, vias 0 -> 6
- net VDD33D: track 31.0 -> 123.7 mm, vias 0 -> 7
- net VDD12A: track 0.00 -> 67.6 mm, vias 0 -> 3
- net Net-(LED1-K): track 1.60 -> 53.0 mm, vias 0 -> 2
- net Net-(LED5-K): track 1.43 -> 44.6 mm, vias 0 -> 2
- net Net-(LED7-K): track 1.60 -> 44.1 mm, vias 0 -> 2
- net VDDAT33: track 12.3 -> 54.7 mm, vias 0 -> 4
- net Net-(LED9-K): track 1.43 -> 40.0 mm, vias 0 -> 2
- net Net-(LED10-K): track 1.53 -> 38.7 mm, vias 0 -> 2
- net SWCLK: track 0.00 -> 35.8 mm, vias 0 -> 1
- net VDD5D: track 15.2 -> 50.7 mm, vias 0 -> 4
- net VDD11D: track 0.44 -> 35.6 mm, vias 0 -> 2
- net Net-(LED8-K): track 1.60 -> 36.2 mm, vias 0 -> 2
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- added copper zone on B.Cu, net GND
- added copper zone on F.Cu, net GND
- added copper zone on B.Cu, net GNDS
Other:
- board size 31 x 100.5 mm -> 31 x 75 mm
