File: zz_micro_l2sw.kicad_sch (KiCad schematic)
At the start: 0 parts

Commit message: modify
Other:
- removed sheet RPico
- removed sheet ksz2pico
- added sheet RPico__ (RPico__.kicad_sch)
Changed lines of the file:
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@@
 	)
 	(sheet
-		(at 226.06 217.17)
-		(size 12.7 19.05)
+		(at 99.06 213.36)
+		(size 22.86 25.4)
 		(exclude_from_sim no)
 		(in_bom yes)
@@
 			(color 0 0 0 0.0000)
 		)
-		(property "Sheetname" "RPico"
-			(at 226.06 216.4584 0)
+		(property "Sheetname" "RPico__"
+			(at 99.06 212.6484 0)
 			(effects
 				(font
@@
 			)
 		)
-		(property "Sheetfile" "RPico.kicad_sch"
-			(at 226.06 236.8046 0)
+		(property "Sheetfile" "RPico__.kicad_sch"
+			(at 99.06 239.3446 0)
 			(effects
 				(font
@@
 			(project "zz_micro_l2sw"
 				(path "/447897ee-d593-43ec-bbc2-e24b07b28d45"
-					(page "3")
+					(page "7")
 				)
 			)
-		)
-	)
-	(sheet
-		(at 300.99 219.71)
-		(size 12.7 19.05)
-		(exclude_from_sim no)
-		(in_bom yes)
-		(on_board yes)
-		(dnp no)
-		(fields_autoplaced yes)
-		(stroke
-			(width 0.1524)
-			(type solid)
-		)
-		(fill
-			(color 0 0 0 0.0000)
-		)
-		(property "Sheetname" "ksz2pico"
-			(at 300.99 218.9984 0)
-			(effects
-				(font
-					(size 1.27 1.27)
-				)
-				(justify left bottom)
-			)
-		)
-		(property "Sheetfile" "ksz2pico.kicad_sch"
-			(at 300.99 239.3446 0)
-			(effects
-				(font
-					(size 1.27 1.27)
-				)
-				(justify left top)
-			)
-		)
-		(instances
-			(project "zz_micro_l2sw"
-				(path "/447897ee-d593-43ec-bbc2-e24b07b28d45"
-					(page "4")
-				)
-			)
